File: hardware/OPNpool_r5/OPNpool_r5.kicad_sch (KiCad schematic)
At the start: 15 parts, among them J1 TERM_BLOCK, U1 MAX3485

Commit message: rename pins
Connections:
- net +3V3: now also PCB1.J1_1 (3V3); no longer PCB1.3V3
- net GND: now also PCB1.J1_15 (GND), PCB1.J3_1 (GND), PCB1.J3_12 (GND), PCB1.J3_15 (GND); no longer PCB1.GND, PCB1.GND@1 (GND), PCB1.GND@2 (GND), PCB1.GND@3 (GND)
- net RTS1: now also PCB1.J3_5 (RTS1/IO23); no longer PCB1.IO23 (RTS1/IO23)
- net RX1: now also PCB1.J3_7 (RX1/IO21); no longer PCB1.IO21 (RX1/IO21)
- net TX1: now also PCB1.J3_6 (TX1/IO22); no longer PCB1.IO22 (TX1/IO22)
- net at D3.C: now also PCB1.J1_14 (5V0); no longer PCB1.5V0
Other:
- moved on the sheet: J1
